File: components/video-output/schematics/mx01-gpu/board.brd (EAGLE design)
At the start: 87 x 79 mm, 28 parts

Commit message: Finish board v.0.01
Parts:
- moved POWER_OUT 82.3 mm to (48.0, 2.00), turned to 0 degrees
- moved POWER 81.0 mm to (42.0, 2.00), turned to 0 degrees
- moved COLOR_OUT 79.2 mm to (6.00, 44.0)
- moved SHIFT_SLAVE 32.0 mm to (70.0, 49.0)
- moved COLOR_IN 15.7 mm to (2.00, 44.0)
- moved SHIFT_MASTER 7.00 mm to (21.0, 49.0)
- moved ADDRESS_OUT 4.00 mm to (84.0, 58.0)
Other:
- board text removed: "mx01-video-component"
- board text removed: "v0.0.1"
