File: components/video-output/schematics/mx01-gpu/board.sch (EAGLE design)
At the start: 19 parts

Commit message: Finish board v.0.01
Parts:
- removed ARDUINO_NANO1: (no value), ArduinoNanoV30:ARDUINO_NANO
- removed J2, J3, J5, J6: (no value), SparkFun-Connectors:CONN_04
- added ADDRESS_IN, ADDRESS_OUT: (no value), SparkFun-Connectors:CONN_08X2
- added ARD_LFT, ARD_RLT: (no value), SparkFun-Connectors:CONN_15
- added C1: 10nF, SparkFun-Capacitors:10NF-PTH-10MM-10000V-1-%
- added COLOR_OUT: (no value), SparkFun-Connectors:CONN_05
- added POWER, POWER_OUT: (no value), SparkFun-Connectors:CONN_02
- added R6, R7, R8, R9: 10k, SparkFun-Resistors:10KOHM-HORIZ-1/4W-5%
- added SHIFT_MASTER, SHIFT_SLAVE: 4021N, 40xx:4021N
- renumbered J4 to COLOR_IN
Connections:
- removed net N$25: ARDUINO_NANO1.D9/OC1A
- removed net N$26: ARDUINO_NANO1.D10/OC1B/!SS
- removed net N$28: ARDUINO_NANO1.D12/MISO
- new net ADDRESS_BIT0: ADDRESS_IN.16, ADDRESS_OUT.16, SHIFT_SLAVEA.P1
- new net ADDRESS_BIT1: ADDRESS_IN.14, ADDRESS_OUT.14, SHIFT_SLAVEA.P2
- new net ADDRESS_BIT10: ADDRESS_IN.11, ADDRESS_OUT.11, SHIFT_MASTERA.P3
- new net ADDRESS_BIT11: ADDRESS_IN.9, ADDRESS_OUT.9, SHIFT_MASTERA.P4
- new net ADDRESS_BIT12: ADDRESS_IN.7, ADDRESS_OUT.7, SHIFT_MASTERA.P5
- new net ADDRESS_BIT13: ADDRESS_IN.5, ADDRESS_OUT.5, SHIFT_MASTERA.P6
- new net ADDRESS_BIT14: ADDRESS_IN.3, ADDRESS_OUT.3, SHIFT_MASTERA.P7
- new net ADDRESS_BIT15: ADDRESS_IN.1, ADDRESS_OUT.1, SHIFT_MASTERA.P8
- new net ADDRESS_BIT2: ADDRESS_IN.12, ADDRESS_OUT.12, SHIFT_SLAVEA.P3
- new net ADDRESS_BIT3: ADDRESS_IN.10, ADDRESS_OUT.10, SHIFT_SLAVEA.P4
- new net ADDRESS_BIT4: ADDRESS_IN.8, ADDRESS_OUT.8, SHIFT_SLAVEA.P5
- new net ADDRESS_BIT5: ADDRESS_IN.6, ADDRESS_OUT.6, SHIFT_SLAVEA.P6
- new net ADDRESS_BIT6: ADDRESS_IN.4, ADDRESS_OUT.4, SHIFT_SLAVEA.P7
- new net ADDRESS_BIT7: ADDRESS_IN.2, ADDRESS_OUT.2, SHIFT_SLAVEA.P8
- new net ADDRESS_BIT8: ADDRESS_IN.15, ADDRESS_OUT.15, SHIFT_MASTERA.P1
- new net ADDRESS_BIT9: ADDRESS_IN.13, ADDRESS_OUT.13, SHIFT_MASTERA.P2
- new net ADDRESS_CLOCK: ARD_LFT.13, SHIFT_MASTERA.CLK, SHIFT_SLAVEA.CLK
- new net ADDRESS_LATCH: ARD_LFT.15, SHIFT_MASTERA.P/!S, SHIFT_SLAVEA.P/!S
- new net ADDRESS_OUTPUT: ARD_LFT.12, SHIFT_MASTERA.Q8
- new net ADDRESS_SERIAL_INPUT: SHIFT_MASTERA.SI, SHIFT_SLAVEA.Q8
- net 5V: now also ARD_RLT.15, C1.1, POWER.1, POWER_OUT.1, SHIFT_MASTERP.VDD, SHIFT_SLAVEP.VDD; no longer ARDUINO_NANO1.VIN
- net BIT0: now also ARD_RLT.7, COLOR_OUT.4, R9.2; no longer ARDUINO_NANO1.ADC3/A3
- net BIT1: now also ARD_RLT.6, COLOR_OUT.3, R8.2; no longer ARDUINO_NANO1.ADC2/A2
- net BIT2: now also ARD_RLT.5, COLOR_OUT.2, R7.2; no longer ARDUINO_NANO1.ADC1/A1
- net BIT3: now also ARD_RLT.4, COLOR_OUT.1, R6.2; no longer ARDUINO_NANO1.ADC0/A0
- net CS: now also ARD_LFT.11; no longer ARDUINO_NANO1.D8/CLK0
- net DC: now also ARD_LFT.9; no longer ARDUINO_NANO1.D6/AIN0
- net GND: now also ARD_RLT.14, C1.2, POWER.2, POWER_OUT.2, R6.1, R7.1, R8.1, R9.1, SHIFT_MASTERP.VSS, SHIFT_SLAVEP.VSS; no longer ARDUINO_NANO1.GND@2
- net N$1: now also ARD_RLT.9; no longer ARDUINO_NANO1.ADC5/SCL/A5
- net N$11: now also ARD_RLT.3; no longer ARDUINO_NANO1.AREF
- net N$12: now also ARD_RLT.2; no longer ARDUINO_NANO1.3V3
- net N$14: now also ARD_LFT.1; no longer ARDUINO_NANO1.D1/TX
- net N$15: now also ARD_LFT.2; no longer ARDUINO_NANO1.D0/RX
- net N$16: now also ARD_LFT.3; no longer ARDUINO_NANO1.!RESET@1
- net N$17: now also ARD_LFT.4; no longer ARDUINO_NANO1.GND@1
- net N$19: now also ARD_LFT.6; no longer ARDUINO_NANO1.D3/INT1
- net N$2: now also ARD_RLT.8; no longer ARDUINO_NANO1.ADC4/SDA/A4
- net N$20: now also ARD_LFT.7; no longer ARDUINO_NANO1.D4/T0
- net N$21: now also ARD_LFT.8; no longer ARDUINO_NANO1.D5/T1
- net N$3: now also ARD_RLT.13; no longer ARDUINO_NANO1.!RESET@2
- net N$5: now also ARD_RLT.11; no longer ARDUINO_NANO1.ADC7/A7
- net N$6: now also ARD_RLT.10; no longer ARDUINO_NANO1.ADC6/A6
- net RST: now also ARD_LFT.10; no longer ARDUINO_NANO1.D7/AIN1
- net SCK: now also ARD_RLT.1; no longer ARDUINO_NANO1.SCK/D13
- net SI: now also ARD_LFT.14; no longer ARDUINO_NANO1.D11/MOSI
- net VIN5V: now also ARD_RLT.12; no longer ARDUINO_NANO1.5V
- net WRITE_ON: now also ARD_LFT.5, COLOR_OUT.5; no longer ARDUINO_NANO1.D2/INT0
